Commit message: camera 2 finger

File: kinova-ros/kinova_description/urdf/camera.xacro (robot description, xacro)
@@ -2,5 +2,5 @@
 <robot xmlns:xacro="http://www.ros.org/wiki/xacro" >
     <joint name="camera_joint" type="fixed">
-        <parent link="j2n6s300_link_6"/>
+        <parent link="j2n6s200_link_6"/>
         <child link="camera_link"/>
         <origin xyz="0.06 0 0.00" rpy="0 ${pi/2} 0"/>

File: kinova-ros/kinova_description/urdf/j2n6s200.xacro (robot description, xacro)
@@ -16,4 +16,5 @@
     <xacro:include filename="$(find kinova_description)/urdf/kinova_common.xacro" />
     <xacro:include filename="$(find kinova_description)/urdf/kinova_finger_set.xacro" />
+    <xacro:include filename="$(find kinova_description)/urdf/camera.xacro" />
     <!-- Import all Gazebo-customization elements -->
     <xacro:include filename="$(find kinova_description)/urdf/kinova.gazebo" />

Commit message: camera pos

File: kinova-ros/kinova_description/urdf/camera.xacro (robot description, xacro)
@@ -4,5 +4,5 @@
         <parent link="j2n6s200_link_6"/>
         <child link="camera_link"/>
-        <origin xyz="0.06 0 0.00" rpy="0 ${pi/2} 0"/>
+        <origin xyz="0.07 0 0.00" rpy="0 ${pi/2} 0"/>
     </joint>
     <link name="camera_link">
