Commit message: action

File: ros_kortex/kortex_description/arms/gen3/6dof/urdf/gen3_macro.xacro (robot description, xacro)
@@ -245,4 +245,34 @@
         <child  link="${prefix}camera_link" />
       </joint>
+      <joint name="camera_optical_joint" type="fixed">
+          <parent link="${prefix}camera_link"/>
+          <child link="camera_link_optical"/>
+          <origin xyz="0 0 0" rpy="${-pi/2} 0 ${-pi/2}"/>
+      </joint>
+    <link name="camera_link_optical"></link>
+      <gazebo reference="${prefix}camera_link">
+        <material>Gazebo/Red</material>
+        <sensor name="camera" type="camera">
+            <pose> 0 0 0 0 0 0 </pose>
+            <visualize>true</visualize>
+            <update_rate>10</update_rate>
+            <camera>
+                <horizontal_fov>1.089</horizontal_fov>
+                <image>
+                    <format>R8G8B8</format>
+                    <width>640</width>
+                    <height>480</height>
+                </image>
+                <clip>
+                    <near>0.05</near>
+                    <far>8.0</far>
+                </clip>
+            </camera>
+            <plugin name="camera_controller" filename="libgazebo_ros_camera.so">
+                <cameraName>camera</cameraName>
+                <frame_name>camera_link_optical</frame_name>
+            </plugin>
+        </sensor>
+      </gazebo>
       <link name="${prefix}camera_depth_frame" />
       <joint name="${prefix}depth_module" type="fixed">

Commit message: camera

File: ros_kortex/kortex_description/arms/gen3/6dof/urdf/gen3_macro.xacro (robot description, xacro)
@@ -241,5 +241,5 @@
       <link name="${prefix}camera_link" />
       <joint name="${prefix}camera_module" type="fixed">
-        <origin xyz="0 0.05639 -0.00305" rpy="3.14159265358979 3.14159265358979 0" />
+        <origin xyz="0 0.05639 -0.00305" rpy="${pi} ${-pi/2} 0" />
         <parent link="${prefix}end_effector_link" />
         <child  link="${prefix}camera_link" />
@@ -248,9 +248,8 @@
           <parent link="${prefix}camera_link"/>
           <child link="camera_link_optical"/>
-          <origin xyz="0 0 0" rpy="${-pi/2} 0 ${-pi/2}"/>
-      </joint>
-    <link name="camera_link_optical"></link>
+          <origin xyz="0 0 0" rpy="0 0 0"/>
+      </joint>
+      <link name="camera_link_optical"></link>
       <gazebo reference="${prefix}camera_link">
-        <material>Gazebo/Red</material>
         <sensor name="camera" type="camera">
             <pose> 0 0 0 0 0 0 </pose>
@@ -277,5 +276,5 @@
       <link name="${prefix}camera_depth_frame" />
       <joint name="${prefix}depth_module" type="fixed">
-        <origin xyz="0.0275 0.066 -0.00305" rpy="3.14159265358979 3.14159265358979 0" />
+        <origin xyz="0.0275 0.066 -0.00305" rpy="${pi} ${pi} 0" />
         <parent link="${prefix}end_effector_link" />
         <child  link="${prefix}camera_depth_frame" />
@@ -283,5 +282,5 @@
       <link name="${prefix}camera_color_frame" />
       <joint name="${prefix}color_module" type="fixed">
-        <origin xyz="0 0.05639 -0.00305" rpy="3.14159265358979 3.14159265358979 0" />
+        <origin xyz="0 0.05639 -0.00305" rpy="${pi} ${pi} 0" />
         <parent link="${prefix}end_effector_link" />
         <child  link="${prefix}camera_color_frame" />

Commit message: making a task env

File: ros_kortex/kortex_description/arms/gen3/6dof/urdf/gen3_macro.xacro (robot description, xacro)
@@ -255,11 +255,11 @@
             <pose> 0 0 0 0 0 0 </pose>
             <visualize>true</visualize>
-            <update_rate>10</update_rate>
+            <update_rate>30</update_rate>
             <camera>
                 <horizontal_fov>1.089</horizontal_fov>
                 <image>
                     <format>R8G8B8</format>
-                    <width>640</width>
-                    <height>480</height>
+                    <width>1280</width>
+                    <height>720</height>
                 </image>
                 <clip>
@@ -268,7 +268,10 @@
                 </clip>
             </camera>
-            <plugin name="camera_controller" filename="libgazebo_ros_camera.so">
+            <plugin name="camera_plugin" filename="libgazebo_ros_camera.so">
                 <cameraName>camera</cameraName>
+                <alwaysOn>true</alwaysOn>
                 <frame_name>camera_link_optical</frame_name>
+                <imageTopicName>/camera/color/image_raw</imageTopicName>
+                <cameraInfoTopicName>/camera/color/camera_info</cameraInfoTopicName>
             </plugin>
         </sensor>
@@ -280,4 +283,36 @@
         <child  link="${prefix}camera_depth_frame" />
       </joint>
+      <joint name="camera_depth_joint" type="fixed">
+          <parent link="${prefix}camera_depth_frame"/>
+          <child link="camera_link_depth"/>
+          <origin xyz="0 0 0" rpy="0 0 0"/>
+      </joint>
+      <link name="camera_link_depth"></link>
+      <gazebo reference="${prefix}camera_depth_frame">
+        <sensor name="camera" type="depth">
+            <pose> 0 0 0 0 0 0 </pose>
+            <update_rate>30</update_rate>
+            <camera>
+                <horizontal_fov>1.089</horizontal_fov>
+                <image>
+                    <format>R8G8B8</format>
+                    <width>1280</width>
+                    <height>720</height>
+                </image>
+                <clip>
+                    <near>0.05</near>
+                    <far>8.0</far>
+                </clip>
+            </camera>
+            <plugin name="camera_plugin" filename="libgazebo_ros_openni_kinect.so">
+                <cameraName>camera_ir</cameraName>
+                <alwaysOn>true</alwaysOn>
+                <frame_name>camera_link_depth</frame_name>
+                <depthImageTopicName>/camera/depth/image_raw</depthImageTopicName>
+                <depthImageCameraInfoTopicName>/camera/depth/camera_info</depthImageCameraInfoTopicName>
+                <pointCloudTopicName>/camera/depth/points</pointCloudTopicName>
+            </plugin>
+        </sensor>
+      </gazebo>
       <link name="${prefix}camera_color_frame" />
       <joint name="${prefix}color_module" type="fixed">

Commit message: joint data and gave up on depth cam for now

File: ros_kortex/kortex_description/arms/gen3/6dof/urdf/gen3_macro.xacro (robot description, xacro)
@@ -283,36 +283,4 @@
         <child  link="${prefix}camera_depth_frame" />
       </joint>
-      <joint name="camera_depth_joint" type="fixed">
-          <parent link="${prefix}camera_depth_frame"/>
-          <child link="camera_link_depth"/>
-          <origin xyz="0 0 0" rpy="0 0 0"/>
-      </joint>
-      <link name="camera_link_depth"></link>
-      <gazebo reference="${prefix}camera_depth_frame">
-        <sensor name="camera" type="depth">
-            <pose> 0 0 0 0 0 0 </pose>
-            <update_rate>30</update_rate>
-            <camera>
-                <horizontal_fov>1.089</horizontal_fov>
-                <image>
-                    <format>R8G8B8</format>
-                    <width>1280</width>
-                    <height>720</height>
-                </image>
-                <clip>
-                    <near>0.05</near>
-                    <far>8.0</far>
-                </clip>
-            </camera>
-            <plugin name="camera_plugin" filename="libgazebo_ros_openni_kinect.so">
-                <cameraName>camera_ir</cameraName>
-                <alwaysOn>true</alwaysOn>
-                <frame_name>camera_link_depth</frame_name>
-                <depthImageTopicName>/camera/depth/image_raw</depthImageTopicName>
-                <depthImageCameraInfoTopicName>/camera/depth/camera_info</depthImageCameraInfoTopicName>
-                <pointCloudTopicName>/camera/depth/points</pointCloudTopicName>
-            </plugin>
-        </sensor>
-      </gazebo>
       <link name="${prefix}camera_color_frame" />
       <joint name="${prefix}color_module" type="fixed">

Commit message: rotated camera

File: ros_kortex/kortex_description/arms/gen3/6dof/urdf/gen3_macro.xacro (robot description, xacro)
@@ -241,5 +241,5 @@
       <link name="${prefix}camera_link" />
       <joint name="${prefix}camera_module" type="fixed">
-        <origin xyz="0 0.05639 -0.00305" rpy="${pi} ${-pi/2} 0" />
+        <origin xyz="0 0.05639 -0.00305" rpy="${pi} ${-pi/2} ${pi/2}" />
         <parent link="${prefix}end_effector_link" />
         <child  link="${prefix}camera_link" />
