Commit message: overhead camera done and publishing

File: setup/misc/gen3_macro.xacro (robot description, xacro)
@@ -26,4 +26,54 @@
       </collision>
     </link>
+      <link name="${prefix}head_camera_link" />
+      <joint name="${prefix}head_camera_module" type="fixed">
+        <origin xyz="0.75 -.2 1.5" rpy="${pi} ${pi/2} ${pi/2}" />
+        <parent link="${prefix}base_link" />
+        <child  link="${prefix}head_camera_link" />
+      </joint>
+      <joint name="head_camera_optical_joint" type="fixed">
+          <parent link="${prefix}head_camera_link"/>
+          <child link="head_camera_link_optical"/>
+          <origin xyz="0 0 0" rpy="0 0 0"/>
+      </joint>
+      <link name="head_camera_link_optical"></link>
+      <gazebo reference="${prefix}head_camera_link">
+        <sensor name="head_camera" type="camera">
+            <pose> 0 0 0 0 0 0 </pose>
+            <visualize>true</visualize>
+            <update_rate>30</update_rate>
+            <camera>
+                <horizontal_fov>1.089</horizontal_fov>
+                <image>
+                    <format>R8G8B8</format>
+                    <width>1280</width>
+                    <height>720</height>
+                </image>
+                <clip>
+                    <near>0.05</near>
+                    <far>8.0</far>
+                </clip>
+            </camera>
+            <plugin name="camera_plugin" filename="libgazebo_ros_camera.so">
+                <cameraName>head_camera</cameraName>
+                <alwaysOn>true</alwaysOn>
+                <frame_name>head_camera_link_optical</frame_name>
+                <imageTopicName>/head_camera/color/image_raw</imageTopicName>
+                <cameraInfoTopicName>/head_camera/color/camera_info</cameraInfoTopicName>
+            </plugin>
+        </sensor>
+      </gazebo>
+      <link name="${prefix}head_camera_depth_frame" />
+      <joint name="${prefix}head_depth_module" type="fixed">
+        <origin xyz="0.0275 0.066 -0.00305" rpy="${pi} ${pi} 0" />
+        <parent link="${prefix}base_link" />
+        <child  link="${prefix}head_camera_depth_frame" />
+      </joint>
+      <link name="${prefix}head_camera_color_frame" />
+      <joint name="${prefix}head_color_module" type="fixed">
+        <origin xyz="0 0.05639 -0.00305" rpy="${pi} ${pi} 0" />
+        <parent link="${prefix}base_link" />
+        <child  link="${prefix}head_camera_color_frame" />
+      </joint>
     <link name="${prefix}shoulder_link">
       <inertial>
